File: boards/0805-phototransistors/readhead-0805.sch (EAGLE design)
At the start: 48 parts

Commit message: new read head board
Parts:
- removed H5, H6, H7, H8: MOUNT-HOLE3.0, holes:MOUNT-HOLE3.0
- added JP3: (no value), pinhead:PINHD-1X4
- added JP4: (no value), pinhead:PINHD-1X8
Connections:
- removed net N$15: R7.2, U$8.E, _1._B6
- removed net N$16: R9.2, U$10.E, _1._B4
- removed net N$17: R8.2, U$9.E, _1._B5
- new net N$18: JP3.1, _1._B3
- new net N$25: JP3.2, _1._B2
- new net N$26: JP3.3, _1._B1
- new net N$27: JP3.4, _1._B0
- new net N$28: JP4.1, _1._B7
- new net N$29: JP4.2, _1._D0
- new net N$30: JP4.3, _1._D1
- new net N$31: JP4.4, _1._D2
- new net N$32: JP4.5, _1._D3
- new net N$33: JP4.6, _1._C6
- new net N$34: JP4.7, _1._C7
- new net N$35: JP4.8, _1._D5
- new net N$36: R7.2, U$8.E, _1._B5
- new net N$37: R8.2, U$9.E, _1._B4
- new net N$38: R9.2, U$10.E, _1._D7
- net N$12: now also _1._F6; no longer _1._F5
- net N$13: now also _1._F7; no longer _1._F6
- net N$14: now also _1._B6; no longer _1._F7
